Commit message: feat(harvest): 스쿱 축방향 삽입 파지 + MoveIt/Nav2 통합 배선 정리
수확 파지 (핵심)
- manipulator_target_node: seat=과실중심(오프셋 0) + 개구축(왼쪽-위) 직선 삽입으로
  전환. 기존 "중심+반경 위 / 수직 CIRC 하강"이 반경만큼 남거나 위로 뜨거나 벽에
  충돌하던 문제 해결. _scoop_insertion_axis(up/left 가중치)로 삽입축 튜닝.
- GRASP/RETRACT_CIRC 모션 CIRC→LIN, seat 정의 3곳(start/refresh/capture) 통일.
- mm_motion_bridge: cmd→MoveGroup 변환, OMPL/Pilz(PTP·LIN·CIRC) 파이프라인.

MoveIt m0617 마이그레이션
- mm_mm URDF/SRDF: Ridgeback+m0617+동축 3축 1/4구 스쿱, harvest_tcp=컵 회전중심.
- moveit_isaac / harvest_pipeline / nav_harvest_pipeline 런치, moveit.rviz.

Nav2 통합
- fleet_dispatch: harvester_nav2 런치 + moveit_nav2 파라미터.

Isaac 측
- mm/harvester_mm/tomato_plants/ripeness/robot_bridge/iw/main 갱신.

기타
- 신규 fixed_harvest_moveit 노드/런치, tools/plot_harvest_tcp_center_path.py.

Co-Authored-By: Claude Opus 4.8 (1M context) <noreply@anthropic.com>

File: src/smartfarm/mm_moveit/urdf/mm_mm.urdf.xacro (robot description, xacro)
@@ -153,22 +153,25 @@
     <hardware>
       <plugin>topic_based_ros2_control/TopicBasedSystem</plugin>
-      <!-- ros2_control_node의 namespace를 따르는 상대 토픽. launch의 ns 인자를
-           바꿔도 하드웨어 채널이 같은 namespace 안에서 함께 이동한다. -->
-      <param name="joint_commands_topic">joint_command</param>
-      <param name="joint_states_topic">hw_joint_states</param>
+      <!-- TopicBasedSystem은 controller_manager와 별도의 내부 노드를 만들기 때문에
+           상대 토픽이 controller_manager의 namespace를 상속하지 않는다. 상대 이름을
+           쓰면 /joint_command·/hw_joint_states를 열어 Isaac의 실제 상태를 못 받고
+           JSB/MoveIt이 0 rad(일자 자세)를 계속 발행한다. Isaac 브리지와 같은 절대
+           하드웨어 채널을 사용한다. -->
+      <param name="joint_commands_topic">/harvester_0/joint_command</param>
+      <param name="joint_states_topic">/harvester_0/hw_joint_states</param>
     </hardware>
     <joint name="joint_1">
-      <command_interface name="position"><param name="initial_value">0.0</param></command_interface>
-      <state_interface name="position"><param name="initial_value">0.0</param></state_interface>
+      <command_interface name="position"><param name="initial_value">3.1415927</param></command_interface>
+      <state_interface name="position"><param name="initial_value">3.1415927</param></state_interface>
       <state_interface name="velocity"/>
     </joint>
     <joint name="joint_2">
-      <command_interface name="position"><param name="initial_value">0.0</param></command_interface>
-      <state_interface name="position"><param name="initial_value">0.0</param></state_interface>
-      <state_interface name="velocity"/>
-    </joint>
-    <joint name="joint_3">
       <command_interface name="position"><param name="initial_value">1.0471976</param></command_interface>
       <state_interface name="position"><param name="initial_value">1.0471976</param></state_interface>
+      <state_interface name="velocity"/>
+    </joint>
+    <joint name="joint_3">
+      <command_interface name="position"><param name="initial_value">-2.0943951</param></command_interface>
+      <state_interface name="position"><param name="initial_value">-2.0943951</param></state_interface>
       <state_interface name="velocity"/>
     </joint>
@@ -179,11 +182,11 @@
     </joint>
     <joint name="joint_5">
-      <command_interface name="position"><param name="initial_value">1.3089969</param></command_interface>
-      <state_interface name="position"><param name="initial_value">1.3089969</param></state_interface>
+      <command_interface name="position"><param name="initial_value">-0.5235988</param></command_interface>
+      <state_interface name="position"><param name="initial_value">-0.5235988</param></state_interface>
       <state_interface name="velocity"/>
     </joint>
     <joint name="joint_6">
-      <command_interface name="position"><param name="initial_value">-1.5707963</param></command_interface>
-      <state_interface name="position"><param name="initial_value">-1.5707963</param></state_interface>
+      <command_interface name="position"><param name="initial_value">1.5707963</param></command_interface>
+      <state_interface name="position"><param name="initial_value">1.5707963</param></state_interface>
       <state_interface name="velocity"/>
     </joint>
